Commit message: Setup visual links at corrected positions

File: robots/hands/leap_hand/leap_hand_right_glb.urdf (robot description, URDF)
Before this commit: robot leap_right, 22 links, 21 joints
Links:
- removed link base
- removed link index_tip_head
- removed link middle_tip_head
- removed link ring_tip_head
- removed link thumb_tip_head
- added link index_finger_dip
- added link index_finger_mcp
- added link index_finger_pip
- added link index_finger_tip
- added link middle_finger_dip
- added link middle_finger_mcp
- added link middle_finger_pip
- added link middle_finger_tip
- added link ring_finger_dip
- added link ring_finger_mcp
- added link ring_finger_pip
- added link ring_finger_tip
- added link thumb_cmc
- added link thumb_ip
- added link thumb_mcp
- added link thumb_tip
- added link wrist
Joints:
- removed joint base_joint
- removed joint index_tip
- removed joint middle_tip
- removed joint ring_tip
- removed joint thumb_tip
- added joint index_finger_dip_joint: type fixed, parent fingertip, child index_finger_dip, origin xyz=0 0 0.014 rpy=0 0 0
- added joint index_finger_mcp_joint: type fixed, parent mcp_joint, child index_finger_mcp, origin xyz=0 0 0.014 rpy=0 0 0
- added joint index_finger_pip_joint: type fixed, parent pip, child index_finger_pip, origin xyz=0.01 0 -0.014 rpy=0 0 0
- added joint index_finger_tip_joint: type fixed, parent fingertip, child index_finger_tip, origin xyz=0 -0.04 0.015 rpy=0 0 0
- added joint middle_finger_dip_joint: type fixed, parent fingertip_2, child middle_finger_dip, origin xyz=0 0 0.014 rpy=0 0 0
- added joint middle_finger_mcp_joint: type fixed, parent mcp_joint_2, child middle_finger_mcp, origin xyz=0 0 0.014 rpy=0 0 0
- added joint middle_finger_pip_joint: type fixed, parent pip_2, child middle_finger_pip, origin xyz=0.01 0 -0.014 rpy=0 0 0
- added joint middle_finger_tip_joint: type fixed, parent fingertip_2, child middle_finger_tip, origin xyz=0 -0.04 0.015 rpy=0 0 0
- added joint ring_finger_dip_joint: type fixed, parent fingertip_3, child ring_finger_dip, origin xyz=0 0 0.014 rpy=0 0 0
- added joint ring_finger_mcp_joint: type fixed, parent mcp_joint_3, child ring_finger_mcp, origin xyz=0 0 0.014 rpy=0 0 0
- added joint ring_finger_pip_joint: type fixed, parent pip_3, child ring_finger_pip, origin xyz=0.01 0 -0.014 rpy=0 0 0
- added joint ring_finger_tip_joint: type fixed, parent fingertip_3, child ring_finger_tip, origin xyz=0 -0.04 0.015 rpy=0 0 0
- added joint thumb_cmc_joint: type fixed, parent thumb_temp_base, child thumb_cmc, origin xyz=0 0 -0.014 rpy=0 0 0
- added joint thumb_ip_joint: type fixed, parent thumb_fingertip, child thumb_ip, origin xyz=0 0 -0.014 rpy=0 0 0
- added joint thumb_mcp_joint: type fixed, parent thumb_dip, child thumb_mcp, origin xyz=0 0 -0.014 rpy=0 0 0
- added joint thumb_tip_joint: type fixed, parent thumb_fingertip, child thumb_tip, origin xyz=0 -0.05 -0.015 rpy=0 0 0
- added joint wrist_joint: type fixed, parent wrist, child palm_lower, origin xyz=0 0.038 0.098 rpy=0 -1.57079 0
